File: pcb/teds-rp2040/teds-rp2040.kicad_pcb (KiCad board)
At the start: 2 copper layers, 21 x 51 mm, 33 parts, among them J1 USB_C_Receptacle_USB2.0_14P, J2 Conn_01x20, J3 Conn_01x20, J4 Conn_01x03, SW1 SW_Push, U1 RP2040, U3 W25Q16JVZPIQ, U4 MCP1700x-330xxTT, Y1 12 MHz

Commit message: Make it work
Parts:
- moved C15 5.73 mm to (41.2, 59.2), turned to -90 degrees
- moved C16 5.70 mm to (35.9, 59.4), turned to 90 degrees
- moved C11 4.71 mm to (43.1, 45.9)
- moved C3 3.41 mm to (41.5, 43.1)
- moved R6 3.10 mm to (37.1, 35.0), turned to 180 degrees
- moved R2 2.86 mm to (38.7, 28.4)
- moved C8 2.79 mm to (42.4, 42.5)
- moved SW1 2.71 mm to (45.4, 33.8)
- moved R1 2.22 mm to (41.6, 28.4)
- moved C6 2.21 mm to (35.1, 52.3)
- moved C5 2.17 mm to (46.2, 52.1)
- moved C2 2.11 mm to (45.5, 46.2), turned to 45 degrees
- moved R7 2.02 mm to (45.5, 37.1)
- moved R5 2.00 mm to (39.5, 57.0)
- moved U1 2.00 mm to (40.3, 51.1)
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Connections:
- Y1 pad 2: XIN -> Net-(C15-Pad2)
- Y1 pad 4: Net-(C15-Pad2) -> XIN
Routing:
- net GND: track 88.9 -> 39.7 mm, vias 13 -> 37
- net GPIO2: track 40.7 -> 24.9 mm
- net +3V3: track 75.4 -> 89.5 mm, vias 6 -> 4
- net +1V1: track 13.8 -> 25.1 mm, vias 2 -> 3
- net QSPI_SD2: track 10.3 -> 21.5 mm
- net QSPI_SS: track 32.4 -> 26.5 mm, vias 3 -> 2
- net Net-(J1-CC1): track 6.84 -> 1.72 mm, vias 2 -> 0
- net SWCLK: track 23.8 -> 19.1 mm
- net RUN: track 16.7 -> 12.9 mm, vias 3 -> 1
- net GPIO17: track 19.0 -> 15.2 mm, vias 1 -> 0
- net GPIO21: track 9.85 -> 6.40 mm, vias 1 -> 0
- net XIN: track 9.76 -> 6.58 mm, vias 2 -> 0
- net GPIO13: track 14.1 -> 11.1 mm
- net Net-(J1-CC2): track 4.72 -> 1.76 mm
- net GPIO14: track 19.1 -> 16.4 mm
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Other:
- board text added: "RP2040 teds.one by Dov"
