File: pcb/teds-rp2040/_autosave-teds-rp2040.kicad_pcb (KiCad board)
At the start: 2 copper layers, 21 x 51 mm, 33 parts, among them J1 USB_C_Receptacle_USB2.0_14P, J2 Conn_01x20, J3 Conn_01x20, J4 Conn_01x03, SW1 SW_Push, U1 RP2040, U3 W25Q16JVZPIQ, U4 MCP1700x-330xxTT, Y1 12 MHz

Commit message: add led
Parts:
- added D1: SK6812MINI, LED_SMD:LED_SK6812MINI_PLCC4_3.5x3.5mm_P1.75mm, F.Cu at (39.7, 64.0)
Connections:
- U1 pad 37: unconnected-(U1-GPIO25-Pad37) -> GPIO25
Routing:
- net GPIO25: track 0.00 -> 15.9 mm, vias 0 -> 2
- net +3V3: track 89.5 -> 97.3 mm, vias 4 -> 6
- net GND: track 39.7 -> 45.2 mm
- net GPIO24: track 31.0 -> 36.4 mm
- net +1V1: track 25.1 -> 22.3 mm
- net SWD: track 18.1 -> 15.4 mm
- net GPIO23: track 26.9 -> 27.6 mm
