File: pcb/teds-rp2040/teds-rp2040.kicad_sch (KiCad schematic)
At the start: 33 parts, among them J1 USB_C_Receptacle_USB2.0_14P, J2 Conn_01x20, J3 Conn_01x20, J4 Conn_01x03, SW1 SW_Push, U1 RP2040, U3 W25Q16JVZPIQ, U4 MCP1700x-330xxTT, Y1 12 MHz

Commit message: Make it work
Connections:
- net XIN: now also Y1.4; no longer Y1.2
- net at C15.2, R5.1: now also Y1.2; no longer Y1.4
Other:
- moved on the sheet: Y1
Changed lines of the file:
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@@
 	(symbol
 		(lib_id "Device:Crystal_GND24")
-		(at 247.65 92.71 0)
+		(at 247.65 92.71 180)
 		(unit 1)
 		(exclude_from_sim no)
@@
 		(dnp no)
 		(property "Reference" "Y1"
-			(at 247.65 82.042 0)
+			(at 247.65 103.378 0)
 			(effects
 				(font
@@
 		)
 		(property "Value" "12 MHz"
-			(at 247.65 84.582 0)
+			(at 247.65 100.838 0)
 			(effects
 				(font

Commit message: add led
Parts:
- added D1: SK6812MINI, LED_SMD:LED_SK6812MINI_PLCC4_3.5x3.5mm_P1.75mm, symbol LED:SK6812MINI
Connections:
- net +3V3: now also D1.4 (VDD)
- net GND: now also D1.2 (VSS)
- net GPIO25: now reaches U1.37 (GPIO25)
- net GPIO25: now also D1.3 (DIN)
- no-connect marks 1 -> 0
Other:
- note added: "LED"
